File: 3rd_year/1st_semester/PAC/01_L_2025_10_01/lab1/lab1.kicad_sch (KiCad schematic)
At the start: 11 parts

Commit message: uncommited
Connections:
- net A: now also R1.2, R2.1, R31.1, R32.1, RTh1.2
Changed lines of the file:
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@@
 	)
 	(label "A"
-		(at 72.39 88.9 0)
+		(at 72.39 90.17 0)
 		(effects
 			(font
@@
 	)
 	(label "B"
-		(at 72.39 105.41 0)
+		(at 72.39 106.68 0)
 		(effects
 			(font
@@
 	)
 	(label "A"
-		(at 72.39 54.61 0)
+		(at 72.39 55.88 0)
 		(effects
 			(font
@@
 	)
 	(label "B"
-		(at 72.39 71.12 0)
+		(at 72.39 72.39 0)
 		(effects
 			(font
