File: 3rd_year/1st_semester/PAC/05_L_2025_10_29/T7/T7.kicad_sch (KiCad schematic)
At the start: 11 parts, among them Q1 2N2222

Commit message: uncommited
Parts:
- C3: value 10uF -> 220uF
Other:
- note added: ".tran 10u 5m 0 10u"
