File: 3rd_year/1st_semester/PAC/03_L_2025_10_15/Tema/Tema.kicad_sch (KiCad schematic)
At the start: 5 parts, among them Q1 2N2222

Commit message: PAC
Connections:
- net C: now reaches Q1.1 (C), R3.2
Other:
- note added: ".TF V(/in) V1"
Changed lines of the file:
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@@
 	(generator_version "9.0")
 	(paper "A4")
+	(text ".TF V(/in) V1"
+		(exclude_from_sim no)
+		(at 228.6 120.142 0)
+		(effects
+			(font
+				(size 1.27 1.27)
+			)
+		)
+	)
 	(junction
 		(at 250.19 110.49)
@@
 		)
 	)
+	(label "C"
+		(at 236.22 81.28 0)
+		(effects
+			(font
+				(size 1.27 1.27)
+			)
+			(justify left bottom)
+		)
+	)
