File: 3rd_year/1st_semester/PAC/06_L_2025_10_05/T9/T9.kicad_sch (KiCad schematic)
At the start: 9 parts, among them U1 LM741

Commit message: uncommited
Parts:
- C1, C2: value 100n -> 100nF
Connections:
- no-connect marks 0 -> 2
Changed lines of the file:
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@@
 		(color 0 0 0 0)
+	)
+	(no_connect
+		(at 165.1 129.54)
+	)
+	(no_connect
+		(at 162.56 129.54)
 	)
 	(wire
@@
 			)
 		)
-		(property "Value" "100n"
+		(property "Value" "100nF"
 			(at 181.61 116.84 90)
 			(effects
@@
 			)
 		)
-		(property "Value" "100n"
+		(property "Value" "100nF"
 			(at 135.89 134.62 90)
 			(effects

Commit message: PAC
Parts:
- C1, C2: value 100nF -> 1.5uF
Changed lines of the file:
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@@
 			)
 		)
-		(property "Value" "100nF"
+		(property "Value" "1.5uF"
 			(at 181.61 116.84 90)
 			(effects
@@
 			)
 		)
-		(property "Value" "100nF"
+		(property "Value" "1.5uF"
 			(at 135.89 134.62 90)
 			(effects
